Commit message: ejercicio 1 acabado

File: ejercicio1/ejercicio1.urdf (robot description, URDF)
Before this commit: robot robot_ej1, 3 links, 2 joints
Links:
- removed link horizontal_link
- removed link vertical_link
- added link body_horizontal_link, mass 2.0; collision box size=0.3 0.1 0.1; visual box size=0.3 0.1 0.1
- added link body_vertical_link, mass 2.0; collision box size=0.1 0.1 0.8; visual box size=0.1 0.1 0.8
- link base_link: mass None -> 1.0; geometry collision box size=0.4 0.4 0.2; visual box size=0.4 0.4 0.2
Joints:
- removed joint base_to_horizontal
- removed joint horizontal_to_vertical
- added joint base_to_vertical: type revolute, parent base_link, child body_vertical_link, origin xyz=0 0 0.2, axis 0 1 0, limit lower=-1.5708 upper=1.5708 effort=10.0 velocity=1.0
- added joint vertical_to_horizontal: type revolute, parent body_vertical_link, child body_horizontal_link, origin xyz=0 0 0.8, axis 0 0 1, limit lower=-3.1416 upper=3.1416 effort=10.0 velocity=1.0
